File: kicad/eosEncoderBoard.kicad_pcb (KiCad board)
At the start: 2 copper layers, 72 parts, among them J1 USB_C_Receptacle_USB2.0_16P, J2 DEBUG, J3 EXTRA, SW1 RotaryEncoder, SW10 SHUTTER, SW11 SW_Push, SW2 RotaryEncoder, SW3 RotaryEncoder, SW4 RotaryEncoder, SW5 INTENS, SW6 FORM, SW7 FOCUS, SW8 IMAGE, SW9 COLOR, U1 STM32L072CZT6TR, U2 PCA9548ADB, U3 TPS62A01DRLR, Y1 OSC16M-3.3I/S3T

Commit message: pcb started kinda
Parts:
- C1, C10, C2, C3, C4, C5, C6, C7, C8, C9, D7, L1, R1, R10, R11, R12, R13, R14, R15, R16, R17, R18, R19, R2, R20, R21, R22, R23, R24, R25, R28, R29, R3, R30, R31, R32, R4, R5, R6, R7, R8, R9, U1, U2, U3, Y1: moved to B.Cu
- SW2, SW3, SW4: footprint Rotary_Encoder:RotaryEncoder_Alps_EC11E-Switch_Vertical_H20mm_MountingHoles -> Rotary_Encoder:RotaryEncoder_Alps_EC11E-Switch_Vertical_H20mm
- moved R11 51.4 mm to (145.4, 105.8), turned to 180 degrees
- moved R14 51.4 mm to (145.4, 113.3), turned to 180 degrees
- moved R10 51.4 mm to (145.4, 103.2), turned to 180 degrees
- moved R12 51.4 mm to (145.4, 108.3), turned to 180 degrees
- moved R13 51.4 mm to (145.4, 110.8), turned to 180 degrees
- moved R15 51.4 mm to (145.4, 115.8), turned to 180 degrees
- moved R16 51.4 mm to (145.4, 118.3), turned to 180 degrees
- moved R17 51.4 mm to (145.4, 120.8), turned to 180 degrees
- moved R9 51.4 mm to (145.4, 100.7), turned to 180 degrees
- moved R18 45.3 mm to (141.4, 100.7), turned to 180 degrees
- moved R19 45.3 mm to (141.4, 103.2), turned to 180 degrees
- moved U2 41.5 mm to (138.6, 111.1), turned to 180 degrees
- moved DP1 39.5 mm to (41.1, 83.8)
- moved DP4 37.7 mm to (169.4, 85.1)
- moved DP2 36.3 mm to (80.8, 83.6)
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Other:
- board outline added: 235 x 45 mm
- board text added: "TO DO: Finish Rough encoder/display layout figure out how cherry mx switches work & lay them out update onshape once you figure it out rough placement for like everything else verify reasonable pin assignments for the things that can move on the uC Place USB-C connector with 1.5mm of overhang (guys it's intentional i promise) routing! (boy i hope this can stay as a 2 layer board)"

Commit message: pcb layout done, still need to handle silkscreen and add mounting holes and such
Parts:
- D7: moved to F.Cu
- J1, R26, R27: moved to B.Cu
- J3: footprint Connector_PinSocket_2.54mm:PinSocket_1x06_P2.54mm_Vertical -> Connector_PinSocket_2.54mm:PinSocket_1x05_P2.54mm_Vertical
- SW10, SW5, SW6, SW7, SW8, SW9: footprint Button_Switch_Keyboard:SW_Cherry_MX_1.00u_PCB -> SwitchLED:SW_Cherry_MX_1.00u_PCB_LED0603
- moved D2 60.0 mm to (217.9, 77.0), turned to 180 degrees
- moved J2 57.9 mm to (229.4, 93.0), turned to -90 degrees
- moved R21 54.0 mm to (221.4, 77.0), turned to 0 degrees
- moved SW10 53.9 mm to (253.5, 87.1), turned to 180 degrees
- moved SW6 53.7 mm to (215.4, 87.1), turned to 180 degrees
- moved SW8 53.7 mm to (234.5, 87.1), turned to 180 degrees
- moved D1 50.2 mm to (217.9, 58.0), turned to 180 degrees
- moved SW9 50.0 mm to (253.5, 68.1), turned to 180 degrees
- moved SW5 49.8 mm to (215.4, 68.1), turned to 180 degrees
- moved SW7 49.7 mm to (234.5, 68.1), turned to 180 degrees
- moved C9 48.4 mm to (261.5, 68.7), turned to 0 degrees
- moved J3 47.7 mm to (212.9, 92.9), turned to -90 degrees
- moved R17 47.1 mm to (166.7, 78.8), turned to 90 degrees
- moved C10 43.8 mm to (261.2, 72.5), turned to 0 degrees
- moved D4 43.6 mm to (237.0, 77.0), turned to 180 degrees
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Connections:
- J3 pad 5: EXTRA4 -> GND
- R10 pad 2: SDA1 -> SDA4
- R11 pad 2: SCL2 -> SCL3
- R12 pad 2: SDA2 -> SDA3
- R13 pad 1: SCL3 -> +3.3V
- R13 pad 2: +3.3V -> SCL1
- R14 pad 1: SDA3 -> +3.3V
- R14 pad 2: +3.3V -> SDA1
- R15 pad 1: SCL4 -> +3.3V
- R15 pad 2: +3.3V -> SCL2
- R16 pad 1: SDA4 -> +3.3V
- R16 pad 2: +3.3V -> SDA2
- R9 pad 2: SCL1 -> SCL4
- U1 pad 10: A2 -> B1
- U1 pad 11: B2 -> A1
- U1 pad 12: A3 -> B2
- U1 pad 13: B3 -> A2
- U1 pad 16: A1 -> B3
- U1 pad 17: B1 -> A3
- U1 pad 20: BTN_INTENS -> unconnected-(U1-PB2-Pad20)
- U1 pad 38: EXTRA4 -> BTN_INTENS
- U2 pad 10: SDA4 -> unconnected-(U2-SD3-Pad10)
- U2 pad 11: SCL4 -> unconnected-(U2-SC3-Pad11)
- U2 pad 13: unconnected-(U2-SD4-Pad13) -> SDA1
- U2 pad 14: unconnected-(U2-SC4-Pad14) -> SCL1
- U2 pad 17: unconnected-(U2-SD6-Pad17) -> SDA2
- U2 pad 18: unconnected-(U2-SC6-Pad18) -> SCL2
- U2 pad 4: SDA1 -> SDA4
- U2 pad 5: SCL1 -> SCL4
- U2 pad 6: SDA2 -> unconnected-(U2-SD1-Pad6)
- U2 pad 7: SCL2 -> unconnected-(U2-SC1-Pad7)
- Y1 pad 1: (no net) -> unconnected-(Y1-Pad1)
Routing:
- net +3.3V: track 0.00 -> 558.7 mm, vias 0 -> 12
- net A1: track 0.00 -> 166.1 mm
- net B1: track 0.00 -> 165.0 mm
- net SW1: track 0.00 -> 143.1 mm, vias 0 -> 2
- net SCL1: track 0.00 -> 129.3 mm
- net SDA1: track 0.00 -> 126.6 mm
- net B2: track 0.00 -> 118.0 mm
- net A2: track 0.00 -> 117.5 mm
- net GND: track 0.00 -> 100.9 mm, vias 0 -> 15
- net SW2: track 0.00 -> 96.6 mm
- net SCL2: track 0.00 -> 86.2 mm
- net SDA2: track 0.00 -> 84.5 mm
- net A3: track 0.00 -> 71.8 mm
- net D+: track 0.00 -> 70.6 mm
- net D-: track 0.00 -> 70.5 mm
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- added copper zone on B.Cu, net +3.3V
- added copper zone on B.Cu, net GND
- added copper zone on F.Cu, net GND
Other:
- board text added: "TO DO: figure out how cherry mx switches work & lay them out update onshape once you figure it out rough placement for like everything else verify reasonable pin assignments for the things that can move on the uC Place USB-C connector with 1.5mm of overhang (guys it's intentional i promise) routing! (boy i hope this can stay as a 2 layer board)"
- board text removed: "TO DO: Finish Rough encoder/display layout figure out how cherry mx switches work & lay them out update onshape once you figure it out rough placement for like everything else verify reasonable pin assignments for the things that can move on the uC Place USB-C connector with 1.5mm of overhang (guys it's intentional i promise) routing! (boy i hope this can stay as a 2 layer board)"

Commit message: pcb done other than silkscreen
Parts:
- DP1, DP2, DP3, DP4: footprint Connector_PinSocket_2.54mm:PinSocket_1x04_P2.54mm_Vertical -> Connector_PinHeader_2.54mm:PinHeader_1x04_P2.54mm_Vertical
- SW10, SW5, SW6, SW7, SW8, SW9: footprint SwitchLED:SW_Cherry_MX_1.00u_PCB_LED0603 -> SwitchLED:SW_Cherry_MX_PCB_1.00u_LED0603
- moved J2 12.7 mm to (216.7, 93.0), turned to 90 degrees
- moved J3 10.2 mm to (202.7, 92.9), turned to 90 degrees
- moved SW9 5.68 mm to (256.1, 63.0)
- moved SW10 5.68 mm to (256.1, 82.0)
- moved SW5 5.68 mm to (217.9, 63.0)
- moved SW7 5.68 mm to (237.0, 63.0)
- moved SW6 5.68 mm to (217.9, 82.0)
- moved SW8 5.68 mm to (237.0, 82.0)
- moved R10 3.13 mm to (162.3, 85.7), turned to 0 degrees
- moved R9 2.38 mm to (161.4, 87.2), turned to 0 degrees
- moved R25 0.91 mm to (260.6, 77.3)
- moved R31 0.91 mm to (263.9, 77.3)
- moved R32 0.91 mm to (262.2, 77.3)
- moved SW11 0.45 mm to (206.9, 87.7)
- renumbered R29 to RFB1, R30 to RFB2, R26 to RUSB1, R27 to RUSB2
Connections:
- J2 pad 1: +3.3V -> GND
- J2 pad 2: SWDIO -> BOOT0
- J2 pad 3: SWCLK -> ~{RST}
- J2 pad 4: ~{RST} -> SWCLK
- J2 pad 5: BOOT0 -> SWDIO
- J2 pad 6: GND -> +3.3V
- J3 pad 1: +3.3V -> GND
- J3 pad 2: EXTRA1 -> EXTRA3
- J3 pad 4: EXTRA3 -> EXTRA1
- J3 pad 5: GND -> +3.3V
Routing:
- net BTN_SHUTTER: track 54.8 -> 62.2 mm, vias 0 -> 1
- net BTN_COLOR: track 55.2 -> 62.6 mm
- net BTN_INTENS: track 16.3 -> 23.7 mm
- net BTN_FOCUS: track 35.5 -> 42.9 mm
- net BTN_IMAGE: track 35.4 -> 41.8 mm
- net +3.3V: track 558.7 -> 552.9 mm, vias 12 -> 14
- net BTN_FORM: track 16.1 -> 21.4 mm
- net SDA4: track 12.2 -> 9.12 mm
- net GND: track 100.9 -> 103.6 mm, vias 15 -> 22
- net SCL4: track 12.6 -> 11.2 mm
- net Net-(D7-K): track 4.43 -> 5.28 mm
- net RST: track 38.7 -> 39.3 mm
Other:
- outline, holes or cut-outs redrawn
- board text added: "COLOR"
- board text added: "Computer Goes Here -->"
- board text added: "DEBUG"
- board text added: "ETC Eos #lighthack Encoders"
- board text added: "FOCUS"
- board text added: "FORM"
- board text added: "IMAGE"
- board text added: "INTENS"
- board text added: "Nic DeBruin 2026 ndebruin.com"
- board text added: "PAN"
- board text added: "Power"
- board text added: "RESET"
- board text added: "SHUTTER"
- board text added: "TILT"
- board text added: "Wheel 1"
- board text added: "Wheel 2"
- board text added: "Wheel 3"
- board text added: "Wheel 4"

Commit message: i can't measure
Parts:
- moved SW3 1.33 mm to (135.2, 60.5)
- moved SW4 1.33 mm to (180.2, 60.5)
- moved SW2 1.33 mm to (90.2, 60.5)
- moved SW1 1.32 mm to (45.2, 60.5)
Routing:
- net SW3: track 51.1 -> 49.7 mm
- net SW2: track 96.6 -> 95.3 mm
- net SW1: track 143.1 -> 141.8 mm
- net B2: track 118.0 -> 116.9 mm
- net A4: track 36.8 -> 37.5 mm
- net A2: track 117.5 -> 116.9 mm
- net B1: track 165.0 -> 164.5 mm
Other:
- outline, holes or cut-outs redrawn
